File: Test PCB 1.sch (KiCad schematic (older format))
At the start: 14 parts

Commit message: created a bunch more shit that isn't the feking MCU
Parts:
- added D? (x4): SOD-123, symbol Device:D_Small
- added F?: Polyfuse, symbol Device:Polyfuse
- added MX? (x4): MX-NoLED, symbol MX_Alps_Hybrid:MX-NoLED
- added USB?: Molex-0548190589, symbol random-keyboard-parts:Molex-0548190589
Connections:
- net +5V: now also F?.1
- net D+: now also USB?.3 (D+)
- net D-: now also USB?.4 (D-)
- net GND: now also USB?.1 (GND)
- new net: D?.2 (A), MX?.2 (ROW) (x4)
- new net VCC: F?.2, USB?.5 (VBUS)
Other:
- moved on the sheet: C?, R?, SW?, U?, Y?

Commit message: finished the schematic(for now)
Parts:
- C1, C2, C3, C4, C5, C6, C7: renamed from C?; footprint (none) -> Capacitor_SMD:C_0805_2012Metric
- D1, D2, D3, D4: renamed from D?; footprint (none) -> Diode_SMD:D_SOD-123
- F1: renamed from F?; footprint (none) -> Fuse:Fuse_1206_3216Metric
- MX1, MX2, MX3, MX4: renamed from MX?; footprint (none) -> MX_Alps_Hybrid:MX-1U-NoLED
- R1, R2, R3, R4: renamed from R?; footprint (none) -> Resistor_SMD:R_0805_2012Metric
- SW1: renamed from SW?; footprint (none) -> random-keyboard-parts:SKQG-1155865
- USB1: renamed from USB?; footprint (none) -> random-keyboard-parts:Molex-0548190589
- Y1: renamed from Y?; footprint (none) -> Crystal:Crystal_SMD_3225-4Pin_3.2x2.5mm
- gave numbers to parts that had none: 1
